Commit message: Update DreamWaQ inspired by Metarobotics

File: legged_gym/resources/robots/go2w/urdf/go2w.urdf (robot description, URDF)
Before this commit: robot go2w_description, 33 links, 32 joints
Links:
- link FL_foot: geometry collision cylinder length=0.045 radius=0.086; visual mesh filename=../dae/left_wheel.dae
- link FR_foot: geometry collision cylinder length=0.045 radius=0.086; visual mesh filename=../dae/right_wheel.dae
- link RL_foot: geometry collision cylinder length=0.045 radius=0.086; visual mesh filename=../dae/left_wheel.dae
- link RR_foot: geometry collision cylinder length=0.045 radius=0.086; visual mesh filename=../dae/right_wheel.dae
